File: Microcontroller.sch (KiCad schematic (older format))
At the start: 23 parts

Commit message: changed the MCU to MK20DX256VLH7
-changed the MCU to MK20DX256VLH7
-This branch is deprciated as I am changing back to the K66 series MCU
Parts:
- C16, C19, C20, C21, C22, C23, C24, C25: renamed from C?; footprint (none) -> Capacitors_SMD:C_0402
- C17, C18, C26: renamed from C?; footprint (none) -> micromouse:C_0603
- J1: renamed from J?; footprint (none) -> micromouse:USB_Micro-B
- L2, L3: renamed from L?; footprint (none) -> micromouse:C_0402
- R31, R32, R33: renamed from R?; footprint (none) -> micromouse:C_0402
- U1: renamed from U?; footprint (none) -> micromouse:MKL02Z32VFG4
- U4: renamed from U?; footprint (none) -> micromouse:LP38691
- U5: renamed from U?; footprint QFP50P1200X1200X160-64N -> micromouse:LQFP-64
- Y1: renamed from Y?; footprint (none) -> micromouse:16Mhz_crystal
- s1: renamed from s?; footprint (none) -> micromouse:Switch_teensy
- gave numbers to parts that had none: 1
