File: IR Emitter .sch (KiCad schematic (older format))
At the start: 24 parts, among them Q1 Q_NMOS_DGS, Q2 Q_NMOS_DGS, Q3 Q_NMOS_DGS, Q4 Q_NMOS_DGS, Q5 Q_NMOS_DGS, Q6 Q_NMOS_DGS

Commit message: Rev 1.0 done
Parts:
- C30, C31, C6, C7, C8, C9: manf# (none) -> NONE
- D10, D11, D12, D13, D8, D9: value IRL81A -> (none)
- R15, R16, R17, R18, R19, R20: manf# (none) -> ERJ-2BQFR75X
Connections:
- net LD_EMITTER: now also Q3.2 (G); no longer Q6.2 (G)
- net LF_EMITTER: now also Q1.2 (G); no longer Q4.2 (G)
- net L_EMITTER: now also Q2.2 (G); no longer Q1.2 (G)
- net RD_EMITTER: now also Q4.2 (G); no longer Q2.2 (G)
- net RF_EMITTER: now also Q6.2 (G); no longer Q3.2 (G)
Changed lines of the file:
@@
 P 3475 3450
 F 0 "D9" H 3495 3520 50  0000 L CNN
-F 1 "IRL81A" H 3435 3340 50  0000 C CNN
+F 1 "" H 3435 3340 50  0000 C CNN
 F 2 "micromouse:IR_Emitter" H 3475 3625 50  0001 C CNN
 F 3 "" H 3425 3450 50  0000 C CNN
@@
 P 5000 3425
 F 0 "D10" H 5020 3495 50  0000 L CNN
-F 1 "IRL81A" H 4960 3315 50  0000 C CNN
+F 1 "" H 4960 3315 50  0000 C CNN
 F 2 "micromouse:IR_Emitter" H 5000 3600 50  0001 C CNN
 F 3 "" H 4950 3425 50  0000 C CNN
@@
 P 5700 3425
 F 0 "D11" H 5720 3495 50  0000 L CNN
-F 1 "IRL81A" H 5660 3315 50  0000 C CNN
+F 1 "" H 5660 3315 50  0000 C CNN
 F 2 "micromouse:IR_Emitter" H 5700 3600 50  0001 C CNN
 F 3 "" H 5650 3425 50  0000 C CNN
@@
 P 7200 3425
 F 0 "D12" H 7220 3495 50  0000 L CNN
-F 1 "IRL81A" H 7160 3315 50  0000 C CNN
+F 1 "" H 7160 3315 50  0000 C CNN
 F 2 "micromouse:IR_Emitter" H 7200 3600 50  0001 C CNN
 F 3 "" H 7150 3425 50  0000 C CNN
@@
 F 2 "micromouse:C_0402" V 2780 4075 50  0001 C CNN
 F 3 "" H 2850 4075 50  0001 C CNN
+F 4 "ERJ-2BQFR75X" H 2930 4175 50  0001 C CNN "manf#"
 	1    2850 4075
 	-1   0    0    1
@@
 F 2 "micromouse:C_0402" V 3405 4075 50  0001 C CNN
 F 3 "" H 3475 4075 50  0001 C CNN
+F 4 "ERJ-2BQFR75X" H 3555 4175 50  0001 C CNN "manf#"
 	1    3475 4075
 	-1   0    0    1
@@
 F 2 "micromouse:C_0402" V 4930 4075 50  0001 C CNN
 F 3 "" H 5000 4075 50  0001 C CNN
+F 4 "ERJ-2BQFR75X" H 5080 4175 50  0001 C CNN "manf#"
 	1    5000 4075
 	-1   0    0    1
@@
 F 2 "micromouse:C_0402" V 5630 4050 50  0001 C CNN
 F 3 "" H 5700 4050 50  0001 C CNN
+F 4 "ERJ-2BQFR75X" H 5780 4150 50  0001 C CNN "manf#"
 	1    5700 4050
 	-1   0    0    1
@@
 F 2 "micromouse:C_0402" V 7130 4075 50  0001 C CNN
 F 3 "" H 7200 4075 50  0001 C CNN
+F 4 "ERJ-2BQFR75X" H 7280 4175 50  0001 C CNN "manf#"
 	1    7200 4075
 	-1   0    0    1
@@
 F 2 "micromouse:C_0402" V 7705 4075 50  0001 C CNN
 F 3 "" H 7775 4075 50  0001 C CNN
+F 4 "ERJ-2BQFR75X" H 7855 4175 50  0001 C CNN "manf#"
 	1    7775 4075
 	-1   0    0    1
@@
 P 2850 3450
 F 0 "D8" H 2870 3520 50  0000 L CNN
-F 1 "IRL81A" H 2810 3340 50  0000 C CNN
+F 1 "" H 2810 3340 50  0000 C CNN
 F 2 "micromouse:IR_Emitter" H 2850 3625 50  0001 C CNN
 F 3 "" H 2800 3450 50  0000 C CNN
@@
 P 7775 3425
 F 0 "D13" H 7795 3495 50  0000 L CNN
-F 1 "IRL81A" H 7735 3315 50  0000 C CNN
+F 1 "" H 7735 3315 50  0000 C CNN
 F 2 "micromouse:IR_Emitter" H 7775 3600 50  0001 C CNN
 F 3 "" H 7725 3425 50  0000 C CNN
@@
 F 2 "Capacitors_SMD:C_0603" H 6338 3350 50  0001 C CNN
 F 3 "" H 6300 3500 50  0001 C CNN
+F 4 "NONE" H 6325 3700 50  0001 C CNN "manf#"
 	1    6300 3500
 	1    0    0    -1
@@
 F 2 "Capacitors_SMD:C_0603" H 6738 3350 50  0001 C CNN
 F 3 "" H 6700 3500 50  0001 C CNN
+F 4 "NONE" H 6725 3700 50  0001 C CNN "manf#"
 	1    6700 3500
 	1    0    0    -1
@@
 F 2 "Capacitors_SMD:C_0603" H 4038 3350 50  0001 C CNN
 F 3 "" H 4000 3500 50  0001 C CNN
+F 4 "NONE" H 4025 3700 50  0001 C CNN "manf#"
 	1    4000 3500
 	1    0    0    -1
@@
 F 2 "Capacitors_SMD:C_0603" H 4438 3350 50  0001 C CNN
 F 3 "" H 4400 3500 50  0001 C CNN
+F 4 "NONE" H 4425 3700 50  0001 C CNN "manf#"
 	1    4400 3500
 	1    0    0    -1
 $EndComp
-Wire Wire Line
-	2850 3650 2850 3925
-Wire Wire Line
-	3475 3925 3475 3650
-Wire Wire Line
-	4000 3650 4400 3650
-Wire Wire Line
-	4000 3350 4400 3350
-Wire Wire Line
-	6300 3350 6700 3350
-Wire Wire Line
-	6300 3650 6700 3650
-$Comp
-L GNDD #PWR014
+$Comp
+L GNDD #PWR018
 U 1 1 5946214E
 P 4200 3700
-F 0 "#PWR014" H 4200 3450 50  0001 C CNN
+F 0 "#PWR018" H 4200 3450 50  0001 C CNN
 F 1 "GNDD" H 4200 3550 50  0000 C CNN
 F 2 "" H 4200 3700 50  0001 C CNN
@@
 	1    0    0    -1
 $EndComp
-Wire Wire Line
-	2850 2925 2850 3350
-Wire Wire Line
-	2850 2925 8275 2925
-Wire Wire Line
-	7775 2925 7775 3325
-Wire Wire Line
-	3475 3350 3475 2925
-Connection ~ 3475 2925
-Wire Wire Line
-	5000 2400 5000 3325
-Connection ~ 5000 2925
-Wire Wire Line
-	4200 3350 4200 2925
-Connection ~ 4200 2925
-Connection ~ 4200 3350
-Wire Wire Line
-	5700 3325 5700 2925
-Connection ~ 5700 2925
-Wire Wire Line
-	7200 3325 7200 2925
-Connection ~ 7200 2925
-Wire Wire Line
-	6500 3350 6500 2925
-Connection ~ 6500 2925
-Connection ~ 6500 3350
-Text GLabel 5000 2400 1    59   Input ~ 12
-V2
-Text GLabel 2550 4425 0    39   Input ~ 8
-L_EMITTER
-Text GLabel 3775 4425 2    39   Input ~ 8
-RD_EMITTER
-Text GLabel 4700 4425 0    39   Input ~ 8
-RF_EMITTER
-Text GLabel 6000 4400 2    39   Input ~ 8
-LF_EMITTER
-Text GLabel 6900 4425 0    39   Input ~ 8
-R_EMITTER
-Text GLabel 8075 4425 2    39   Input ~ 8
-LD_EMITTER
-Text Notes 3900 1400 0    394  ~ 79
-IR Emitter
 $Comp
 L C C30
@@
 F 2 "Capacitors_SMD:C_0603" H 8113 3350 50  0001 C CNN
 F 3 "" H 8075 3500 50  0001 C CNN
+F 4 "NONE" H 8100 3700 50  0001 C CNN "manf#"
 	1    8075 3500
 	1    0    0    -1
@@
 F 2 "Capacitors_SMD:C_0603" H 8513 3350 50  0001 C CNN
 F 3 "" H 8475 3500 50  0001 C CNN
+F 4 "NONE" H 8500 3700 50  0001 C CNN "manf#"
 	1    8475 3500
 	1    0    0    -1
 $EndComp
-Wire Wire Line
-	8075 3350 8475 3350
-Wire Wire Line
-	8075 3650 8475 3650
-Wire Wire Line
-	8275 2925 8275 3350
-Connection ~ 8275 3350
-Connection ~ 7775 2925
-Wire Wire Line
-	4200 3700 4200 3650
-Connection ~ 4200 3650
-$Comp
-L GNDD #PWR015
+$Comp
+L GNDD #PWR019
 U 1 1 59D9D983
 P 6500 3675
-F 0 "#PWR015" H 6500 3425 50  0001 C CNN
+F 0 "#PWR019" H 6500 3425 50  0001 C CNN
 F 1 "GNDD" H 6500 3525 50  0000 C CNN
 F 2 "" H 6500 3675 50  0001 C CNN
@@
 $EndComp
 $Comp
-L GNDD #PWR016
+L GNDD #PWR020
 U 1 1 59D9DDA3
 P 8300 3675
-F 0 "#PWR016" H 8300 3425 50  0001 C CNN
+F 0 "#PWR020" H 8300 3425 50  0001 C CNN
 F 1 "GNDD" H 8300 3525 50  0000 C CNN
 F 2 "" H 8300 3675 50  0001 C CNN
@@
 	1    0    0    -1
 $EndComp
-Wire Wire Line
-	6500 3675 6500 3650
-Connection ~ 6500 3650
-Wire Wire Line
-	8300 3675 8300 3650
-Connection ~ 8300 3650
-Wire Wire Line
-	5000 3925 5000 3625
-Wire Wire Line
-	5700 3900 5700 3625
-Wire Wire Line
-	7200 3625 7200 3925
-Wire Wire Line
-	7775 3625 7775 3925
 $Comp
 L Q_NMOS_DGS Q2
@@
 $EndComp
 $Comp
-L GNDD #PWR017
+L GNDD #PWR021
 U 1 1 59DA4EAB
 P 7775 4625
-F 0 "#PWR017" H 7775 4375 50  0001 C CNN
+F 0 "#PWR021" H 7775 4375 50  0001 C CNN
 F 1 "GNDD" H 7775 4475 50  0000 C CNN
 F 2 "" H 7775 4625 50  0001 C CNN
@@
 $EndComp
 $Comp
-L GNDD #PWR018
+L GNDD #PWR022
 U 1 1 59DA52BE
 P 7200 4625
-F 0 "#PWR018" H 7200 4375 50  0001 C CNN
+F 0 "#PWR022" H 7200 4375 50  0001 C CNN
 F 1 "GNDD" H 7200 4475 50  0000 C CNN
 F 2 "" H 7200 4625 50  0001 C CNN
@@
 $EndComp
 $Comp
-L GNDD #PWR019
+L GNDD #PWR023
 U 1 1 59DA5311
 P 5700 4600
-F 0 "#PWR019" H 5700 4350 50  0001 C CNN
+F 0 "#PWR023" H 5700 4350 50  0001 C CNN
 F 1 "GNDD" H 5700 4450 50  0000 C CNN
 F 2 "" H 5700 4600 50  0001 C CNN
@@
 $EndComp
 $Comp
-L GNDD #PWR020
+L GNDD #PWR024
 U 1 1 59DA5544
 P 5000 4625
-F 0 "#PWR020" H 5000 4375 50  0001 C CNN
+F 0 "#PWR024" H 5000 4375 50  0001 C CNN
 F 1 "GNDD" H 5000 4475 50  0000 C CNN
 F 2 "" H 5000 4625 50  0001 C CNN
@@
 $EndComp
 $Comp
-L GNDD #PWR021
+L GNDD #PWR025
 U 1 1 59DA55E9
 P 3475 4625
-F 0 "#PWR021" H 3475 4375 50  0001 C CNN
+F 0 "#PWR025" H 3475 4375 50  0001 C CNN
 F 1 "GNDD" H 3475 4475 50  0000 C CNN
 F 2 "" H 3475 4625 50  0001 C CNN
@@
 $EndComp
 $Comp
-L GNDD #PWR022
+L GNDD #PWR026
 U 1 1 59DA587C
 P 2850 4625
-F 0 "#PWR022" H 2850 4375 50  0001 C CNN
+F 0 "#PWR026" H 2850 4375 50  0001 C CNN
 F 1 "GNDD" H 2850 4475 50  0000 C CNN
 F 2 "" H 2850 4625 50  0001 C CNN
@@
 	1    0    0    -1
 $EndComp
+Text GLabel 5000 2400 1    59   Input ~ 12
+V2
+Text GLabel 3775 4425 2    39   Input ~ 8
+L_EMITTER
+Text GLabel 6000 4400 2    39   Input ~ 8
+RD_EMITTER
+Text GLabel 8075 4425 2    39   Input ~ 8
+RF_EMITTER
+Text GLabel 2550 4425 0    39   Input ~ 8
+LF_EMITTER
+Text GLabel 6900 4425 0    39   Input ~ 8
+R_EMITTER
+Text GLabel 4700 4425 0    39   Input ~ 8
+LD_EMITTER
+Text Notes 3900 1400 0    394  ~ 79
+IR Emitter
+Wire Wire Line
+	2850 3650 2850 3925
+Wire Wire Line
+	3475 3925 3475 3650
+Wire Wire Line
+	4000 3650 4400 3650
+Wire Wire Line
+	4000 3350 4400 3350
+Wire Wire Line
+	6300 3350 6700 3350
+Wire Wire Line
+	6300 3650 6700 3650
+Wire Wire Line
+	2850 2925 2850 3350
+Wire Wire Line
+	2850 2925 8275 2925
+Wire Wire Line
+	7775 2925 7775 3325
+Wire Wire Line
+	3475 3350 3475 2925
+Wire Wire Line
+	5000 2400 5000 3325
+Wire Wire Line
+	4200 3350 4200 2925
+Wire Wire Line
+	5700 3325 5700 2925
+Wire Wire Line
+	7200 3325 7200 2925
+Wire Wire Line
+	6500 3350 6500 2925
+Wire Wire Line
+	8075 3350 8475 3350
+Wire Wire Line
+	8075 3650 8475 3650
+Wire Wire Line
+	8275 2925 8275 3350
+Wire Wire Line
+	4200 3700 4200 3650
+Wire Wire Line
+	6500 3675 6500 3650
+Wire Wire Line
+	8300 3675 8300 3650
+Wire Wire Line
+	5000 3925 5000 3625
+Wire Wire Line
+	5700 3900 5700 3625
+Wire Wire Line
+	7200 3625 7200 3925
+Wire Wire Line
+	7775 3625 7775 3925
+Connection ~ 3475 2925
+Connection ~ 5000 2925
+Connection ~ 4200 2925
+Connection ~ 4200 3350
+Connection ~ 5700 2925
+Connection ~ 7200 2925
+Connection ~ 6500 2925
+Connection ~ 6500 3350
+Connection ~ 8275 3350
+Connection ~ 7775 2925
+Connection ~ 4200 3650
+Connection ~ 6500 3650
+Connection ~ 8300 3650
 $EndSCHEMATC
