File: IR Emitter .sch (KiCad schematic (older format))
At the start: 24 parts, among them Q1 Q_NMOS_DGS, Q2 Q_NMOS_DGS, Q3 Q_NMOS_DGS, Q4 Q_NMOS_DGS, Q5 Q_NMOS_DGS, Q6 Q_NMOS_DGS

Commit message: fixed the unconnected teensy bootloader chip
Parts:
- C30, C31, C6, C7, C8, C9: manf# NONE -> DNP
- D10, D11, D12, D13, D8, D9: value (none) -> ~
Changed lines of the file:
@@
 P 3475 3450
 F 0 "D9" H 3495 3520 50  0000 L CNN
-F 1 "" H 3435 3340 50  0000 C CNN
+F 1 "~" H 3435 3340 50  0000 C CNN
 F 2 "micromouse:IR_Emitter" H 3475 3625 50  0001 C CNN
 F 3 "" H 3425 3450 50  0000 C CNN
@@
 P 5000 3425
 F 0 "D10" H 5020 3495 50  0000 L CNN
-F 1 "" H 4960 3315 50  0000 C CNN
+F 1 "~" H 4960 3315 50  0000 C CNN
 F 2 "micromouse:IR_Emitter" H 5000 3600 50  0001 C CNN
 F 3 "" H 4950 3425 50  0000 C CNN
@@
 P 5700 3425
 F 0 "D11" H 5720 3495 50  0000 L CNN
-F 1 "" H 5660 3315 50  0000 C CNN
+F 1 "~" H 5660 3315 50  0000 C CNN
 F 2 "micromouse:IR_Emitter" H 5700 3600 50  0001 C CNN
 F 3 "" H 5650 3425 50  0000 C CNN
@@
 P 7200 3425
 F 0 "D12" H 7220 3495 50  0000 L CNN
-F 1 "" H 7160 3315 50  0000 C CNN
+F 1 "~" H 7160 3315 50  0000 C CNN
 F 2 "micromouse:IR_Emitter" H 7200 3600 50  0001 C CNN
 F 3 "" H 7150 3425 50  0000 C CNN
@@
 P 2850 3450
 F 0 "D8" H 2870 3520 50  0000 L CNN
-F 1 "" H 2810 3340 50  0000 C CNN
+F 1 "~" H 2810 3340 50  0000 C CNN
 F 2 "micromouse:IR_Emitter" H 2850 3625 50  0001 C CNN
 F 3 "" H 2800 3450 50  0000 C CNN
@@
 P 7775 3425
 F 0 "D13" H 7795 3495 50  0000 L CNN
-F 1 "" H 7735 3315 50  0000 C CNN
+F 1 "~" H 7735 3315 50  0000 C CNN
 F 2 "micromouse:IR_Emitter" H 7775 3600 50  0001 C CNN
 F 3 "" H 7725 3425 50  0000 C CNN
@@
 F 2 "Capacitors_SMD:C_0603" H 6338 3350 50  0001 C CNN
 F 3 "" H 6300 3500 50  0001 C CNN
-F 4 "NONE" H 6325 3700 50  0001 C CNN "manf#"
+F 4 "DNP" H 6325 3700 50  0001 C CNN "manf#"
 	1    6300 3500
 	1    0    0    -1
@@
 F 2 "Capacitors_SMD:C_0603" H 6738 3350 50  0001 C CNN
 F 3 "" H 6700 3500 50  0001 C CNN
-F 4 "NONE" H 6725 3700 50  0001 C CNN "manf#"
+F 4 "DNP" H 6725 3700 50  0001 C CNN "manf#"
 	1    6700 3500
 	1    0    0    -1
@@
 F 2 "Capacitors_SMD:C_0603" H 4038 3350 50  0001 C CNN
 F 3 "" H 4000 3500 50  0001 C CNN
-F 4 "NONE" H 4025 3700 50  0001 C CNN "manf#"
+F 4 "DNP" H 4025 3700 50  0001 C CNN "manf#"
 	1    4000 3500
 	1    0    0    -1
@@
 F 2 "Capacitors_SMD:C_0603" H 4438 3350 50  0001 C CNN
 F 3 "" H 4400 3500 50  0001 C CNN
-F 4 "NONE" H 4425 3700 50  0001 C CNN "manf#"
+F 4 "DNP" H 4425 3700 50  0001 C CNN "manf#"
 	1    4400 3500
 	1    0    0    -1
@@
 F 2 "Capacitors_SMD:C_0603" H 8113 3350 50  0001 C CNN
 F 3 "" H 8075 3500 50  0001 C CNN
-F 4 "NONE" H 8100 3700 50  0001 C CNN "manf#"
+F 4 "DNP" H 8100 3700 50  0001 C CNN "manf#"
 	1    8075 3500
 	1    0    0    -1
@@
 F 2 "Capacitors_SMD:C_0603" H 8513 3350 50  0001 C CNN
 F 3 "" H 8475 3500 50  0001 C CNN
-F 4 "NONE" H 8500 3700 50  0001 C CNN "manf#"
+F 4 "DNP" H 8500 3700 50  0001 C CNN "manf#"
 	1    8475 3500
 	1    0    0    -1
