File: Gyro.sch (KiCad schematic (older format))
At the start: 4 parts, among them U31 MPU-6500

Commit message: Rev 1.0 done
Parts:
- C32, C33, C34: manf# (none) -> NONE
- U31: manf# (none) -> MPU-6500
Connections:
- net 3.3V renamed MCUv
Changed lines of the file:
@@
 F 2 "micromouse:MPU-6500" H 6050 3050 60  0001 C CNN
 F 3 "" H 6050 3050 60  0001 C CNN
+F 4 "MPU-6500" H 5325 3225 50  0001 C CNN "manf#"
 	1    5750 3750
 	1    0    0    -1
 $EndComp
-NoConn ~ 5150 3550
-NoConn ~ 5150 3650
-NoConn ~ 5150 3750
-NoConn ~ 5150 3850
-NoConn ~ 5150 3950
-NoConn ~ 5150 4050
-NoConn ~ 6450 3650
-NoConn ~ 6450 3750
-NoConn ~ 6450 3850
-NoConn ~ 6450 3950
-Wire Wire Line
-	6450 3550 6600 3550
-Wire Wire Line
-	6600 3075 6600 3650
-Wire Wire Line
-	5950 3150 5950 3075
-Wire Wire Line
-	5950 3075 6600 3075
-Connection ~ 6600 3550
-NoConn ~ 6050 3150
-NoConn ~ 5850 3150
-NoConn ~ 5550 4450
 $Comp
 L C C34
@@
 F 2 "Capacitors_SMD:C_0603" H 6688 4150 50  0001 C CNN
 F 3 "" H 6650 4300 50  0001 C CNN
+F 4 "NONE" H 6675 4500 50  0001 C CNN "manf#"
 	1    6650 4300
 	1    0    0    -1
@@
 F 2 "Capacitors_SMD:C_0603" H 5888 4825 50  0001 C CNN
 F 3 "" H 5850 4975 50  0001 C CNN
+F 4 "NONE" H 5875 5175 50  0001 C CNN "manf#"
 	1    5850 4975
 	1    0    0    -1
@@
 F 2 "Capacitors_SMD:C_0603" H 5688 4825 50  0001 C CNN
 F 3 "" H 5650 4975 50  0001 C CNN
+F 4 "NONE" H 5675 5175 50  0001 C CNN "manf#"
 	1    5650 4975
 	1    0    0    -1
 $EndComp
-Text GLabel 5650 2875 1    51   Input ~ 0
-SCLK
-Text GLabel 5550 2875 1    51   Input ~ 0
-SDI
 $Comp
-L GNDD #PWR047
+L GNDD #PWR051
 U 1 1 59AB8073
 P 6600 3650
-F 0 "#PWR047" H 6600 3400 50  0001 C CNN
+F 0 "#PWR051" H 6600 3400 50  0001 C CNN
 F 1 "GNDD" H 6600 3500 50  0000 C CNN
 F 2 "" H 6600 3650 50  0001 C CNN
@@
 $EndComp
 $Comp
-L GNDD #PWR048
+L GNDD #PWR052
 U 1 1 59AB8123
 P 5650 5175
-F 0 "#PWR048" H 5650 4925 50  0001 C CNN
+F 0 "#PWR052" H 5650 4925 50  0001 C CNN
 F 1 "GNDD" H 5650 5025 50  0000 C CNN
 F 2 "" H 5650 5175 50  0001 C CNN
@@
 $EndComp
 $Comp
-L GNDD #PWR049
+L GNDD #PWR053
 U 1 1 59AB814A
 P 5850 5175
-F 0 "#PWR049" H 5850 4925 50  0001 C CNN
+F 0 "#PWR053" H 5850 4925 50  0001 C CNN
 F 1 "GNDD" H 5850 5025 50  0000 C CNN
 F 2 "" H 5850 5175 50  0001 C CNN
@@
 	1    0    0    -1
 $EndComp
+$Comp
+L GNDD #PWR054
+U 1 1 59AB8D41
+P 6650 4500
+F 0 "#PWR054" H 6650 4250 50  0001 C CNN
+F 1 "GNDD" H 6650 4350 50  0000 C CNN
+F 2 "" H 6650 4500 50  0001 C CNN
+F 3 "" H 6650 4500 50  0001 C CNN
+	1    6650 4500
+	1    0    0    -1
+$EndComp
+Text GLabel 5650 2875 1    51   Input ~ 0
+SCLK
+Text GLabel 5550 2875 1    51   Input ~ 0
+SDI
+Text GLabel 5750 4525 3    51   Input ~ 0
+SDO
+Text GLabel 6050 4500 3    51   Input ~ 0
+INT
+Text GLabel 5950 4500 3    51   Input ~ 0
+FSYNC
+Text GLabel 5750 2875 1    51   Input ~ 0
+nCS
+Text GLabel 6775 4050 2    60   Input ~ 0
+MCUv
+Wire Wire Line
+	6450 3550 6600 3550
+Wire Wire Line
+	6600 3075 6600 3650
+Wire Wire Line
+	5950 3150 5950 3075
+Wire Wire Line
+	5950 3075 6600 3075
 Wire Wire Line
 	5650 4450 5650 4825
@@
 Wire Wire Line
 	5850 4450 5850 4825
-Text GLabel 5750 4525 3    51   Input ~ 0
-SDO
 Wire Wire Line
 	5750 4450 5750 4525
@@
 Wire Wire Line
 	5650 2875 5650 3150
-Text GLabel 6050 4500 3    51   Input ~ 0
-INT
 Wire Wire Line
 	6050 4450 6050 4500
-Text GLabel 5950 4500 3    51   Input ~ 0
-FSYNC
 Wire Wire Line
 	5950 4450 5950 4500
@@
 Wire Wire Line
 	6650 4050 6650 4150
-$Comp
-L GNDD #PWR050
-U 1 1 59AB8D41
-P 6650 4500
-F 0 "#PWR050" H 6650 4250 50  0001 C CNN
-F 1 "GNDD" H 6650 4350 50  0000 C CNN
-F 2 "" H 6650 4500 50  0001 C CNN
-F 3 "" H 6650 4500 50  0001 C CNN
-	1    6650 4500
-	1    0    0    -1
-$EndComp
 Wire Wire Line
 	6650 4500 6650 4450
-Text GLabel 6775 4050 2    51   Input ~ 0
-3.3V
-Connection ~ 6650 4050
-Text GLabel 5750 2875 1    51   Input ~ 0
-nCS
 Wire Wire Line
 	5750 3150 5750 2875
+Connection ~ 6600 3550
+Connection ~ 6650 4050
+NoConn ~ 5150 3550
+NoConn ~ 5150 3650
+NoConn ~ 5150 3750
+NoConn ~ 5150 3850
+NoConn ~ 5150 3950
+NoConn ~ 5150 4050
+NoConn ~ 6450 3650
+NoConn ~ 6450 3750
+NoConn ~ 6450 3850
+NoConn ~ 6450 3950
+NoConn ~ 6050 3150
+NoConn ~ 5850 3150
+NoConn ~ 5550 4450
 $EndSCHEMATC

Commit message: fixed the unconnected teensy bootloader chip
Parts:
- C32, C33, C34: manf# NONE -> DNP
Changed lines of the file:
@@
 F 2 "Capacitors_SMD:C_0603" H 6688 4150 50  0001 C CNN
 F 3 "" H 6650 4300 50  0001 C CNN
-F 4 "NONE" H 6675 4500 50  0001 C CNN "manf#"
+F 4 "DNP" H 6675 4500 50  0001 C CNN "manf#"
 	1    6650 4300
 	1    0    0    -1
@@
 F 2 "Capacitors_SMD:C_0603" H 5888 4825 50  0001 C CNN
 F 3 "" H 5850 4975 50  0001 C CNN
-F 4 "NONE" H 5875 5175 50  0001 C CNN "manf#"
+F 4 "DNP" H 5875 5175 50  0001 C CNN "manf#"
 	1    5850 4975
 	1    0    0    -1
@@
 F 2 "Capacitors_SMD:C_0603" H 5688 4825 50  0001 C CNN
 F 3 "" H 5650 4975 50  0001 C CNN
-F 4 "NONE" H 5675 5175 50  0001 C CNN "manf#"
+F 4 "DNP" H 5675 5175 50  0001 C CNN "manf#"
 	1    5650 4975
 	1    0    0    -1
