File: Motor Controller.sch (KiCad schematic (older format))
At the start: 22 parts, among them U10 CONN_02X03, U2 DRV8833, U27 Test_Point, U28 Test_Point, U29 Test_Point, U30 Test_Point, U32 Motor_mount, U9 CONN_02X03

Commit message: Rev 1.0 done
Parts:
- removed R30: R, symbol R
- added R32, R33, R34, R35, R36, R41, R42, R43: R, Capacitors_SMD:C_0402, symbol R
- C35: value C -> 2.2uF; manf# (none) -> GRM155R61A225KE95D
- R1, R2, R4: manf# (none) -> MCS04020Z0000ZE000
- R3: footprint Capacitors_SMD:C_0402 -> micromouse:R_0402; manf# (none) -> MCS04020Z0000ZE000
- R5, R6, R7, R8: manf# (none) -> RC0402JR-074K7L
- U10, U9: manf# (none) -> M20-9980346
- U2: manf# GRM188R71E103KA01D -> DRV8833RTYT
- U27, U28, U29, U30: manf# (none) -> RCU-0C
- U32: manf# (none) -> NONE
Connections:
- net GNDD: now also U2.1 (AISEN), U2.4 (BISEN), R32.2, R35.2, R36.2, R43.2
- net L_CH_A: now also R42.2, R43.1; no longer U10.1 (P1)
- net L_CH_B: now also R34.2, R35.1; no longer U10.2 (P2)
- net R_CH_A: now also R32.1, R33.2; no longer U9.1 (P1)
- net R_CH_B: now also R36.1, R41.2; no longer U9.2 (P2)
- new net: R33.1, U9.1 (P1)
- new net: R41.1, U9.2 (P2)
- new net: R34.1, U10.1 (P1)
- new net: R42.1, U10.2 (P2)

Commit message: fixed the unconnected teensy bootloader chip
Parts:
- U32: manf# NONE -> DNP
Changed lines of the file:
@@
 F 2 "micromouse:Motor_mount" H 9275 3550 60  0001 C CNN
 F 3 "" H 9275 3550 60  0001 C CNN
-F 4 "NONE" H 9275 3575 50  0001 C CNN "manf#"
+F 4 "DNP" H 9275 3575 50  0001 C CNN "manf#"
 	1    9275 3550
 	0    1    1    0
