File: Power System.sch (KiCad schematic (older format))
At the start: 30 parts, among them U15 LMZ21701, U16 JST_Connector, U17 Switch_micromouse, U18 LMZ21701, U19 splitter, U24 Test_Point, U25 Test_Point, U26 Test_Point, U4 TPS61222DCK, U7 Test_Point

Commit message: fixed the unconnected teensy bootloader chip
Parts:
- U16, U17, U19: manf# NONE -> DNP
Changed lines of the file:
@@
 F 2 "micromouse:spliter" H 3050 2100 39  0001 C CNN
 F 3 "" H 3050 2100 39  0001 C CNN
-F 4 "NONE" H 3112 2097 50  0001 C CNN "manf#"
+F 4 "DNP" H 3112 2097 50  0001 C CNN "manf#"
 	1    3050 2100
 	0    1    1    0
@@
 F 2 "micromouse:JST_Connector" H 2000 1675 39  0001 C CNN
 F 3 "" H 1750 1775 39  0001 C CNN
-F 4 "NONE" H 1750 1875 50  0001 C CNN "manf#"
+F 4 "DNP" H 1750 1875 50  0001 C CNN "manf#"
 	1    2000 1675
 	1    0    0    -1
@@
 F 2 "micromouse:Switch_battery" H 2925 1700 39  0001 C CNN
 F 3 "" H 2925 1700 39  0001 C CNN
-F 4 "NONE" H 3175 1975 50  0001 C CNN "manf#"
+F 4 "DNP" H 3175 1975 50  0001 C CNN "manf#"
 	1    2925 1700
 	1    0    0    -1
